File: BR-Motor.kicad_sch (KiCad schematic)
At the start: 27 parts, among them J1 22850120ANG1SYA01, J2 Conn_01x02, J3 Conn_01x02, J4 Conn_01x04, J5 Conn_01x02, Q1 SQD50P04-13L_T4GE3, Q2 BSS138, U1 LM340AT

Commit message: Update PDF shematic
Other:
- title: BR-MOTOR : GPIO Sheet -> BR-MOTOR : MAIN Sheet
Changed lines of the file:
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@@
 	(paper "A4")
 	(title_block
-		(title "BR-MOTOR : GPIO Sheet")
+		(title "BR-MOTOR : MAIN Sheet")
 		(date "2025-02-23")
 		(rev "V°1")
@@
 			)
 		)
-		(property "Datasheet" "http://www.st.com/content/ccc/resource/technical/document/datasheet/41/4f/b3/b0/12/d4/47/88/CD00000444.pdf/files/CD00000444.pdf/jcr:content/translations/en.CD00000444.pdf"
+		(property "Datasheet" "https://www.ti.com/lit/ds/symlink/lm340.pdf?ts=1743830389916"
 			(at 101.6 34.29 0)
 			(effects
