File: GPIOSheet.kicad_sch (KiCad schematic)
At the start: 61 parts, among them J10 Conn_01x03, J11 Conn_01x03, J12 Conn_01x06, J13 Conn_01x04, J14 Conn_01x02, J9 Conn_01x02, U5 ACPL-214-500E, U6 ACPL-214-500E, U7 74HC14, U8 ADuM1281

Commit message: Update PDF shematic
Other:
- company: (none) -> MASTODONTE
Changed lines of the file:
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@@
 		(date "2025-02-23")
 		(rev "V°1")
+		(company "MASTODONTE")
+		(comment 1 "Paul Miailhe")
 	)
 	(junction
@@
 		)
 	)
-	(text_box "ACPL-214 AC Input, Half-Pitch Phototransistor Optocoupler Data Sheet\n- Current transfer ratio (CTR: min. 20% at IF = ±5mA, VCC = 5V)\n- High input-output isolation voltage (VISO = 3,000VRMS)\n- Non-saturated Response time (tr: typ. 2μs at VCC = 10V, IC = 2mA, RL= 100Ω)\n- CMR 10 kV/μs (typical)"
+	(text_box "ACPL-214 AC / TLP292(TPL,E Input, Half-Pitch Phototransistor Optocoupler Data Sheet\n- Current transfer ratio (CTR: min. 20% at IF = ±5mA, VCC = 5V)\n- High input-output isolation voltage (VISO = 3,000VRMS)\n- Non-saturated Response time (tr: typ. 2μs at VCC = 10V, IC = 2mA, RL= 100Ω)\n- CMR 10 kV/μs (typical)"
 		(exclude_from_sim no)
 		(at 213.36 62.23 0)
@@
 		)
 	)
-	(text_box "ACPL-214 AC Input, Half-Pitch Phototransistor Optocoupler Data Sheet\n- Current transfer ratio (CTR: min. 20% at IF = ±5mA, VCC = 5V)\n- High input-output isolation voltage (VISO = 3,000VRMS)\n- Non-saturated Response time (tr: typ. 2μs at VCC = 10V, IC = 2mA, RL= 100Ω)\n- CMR 10 kV/μs (typical)"
+	(text_box "ACPL-214 AC / TLP292(TPL,E Input, Half-Pitch Phototransistor Optocoupler Data Sheet\n- Current transfer ratio (CTR: min. 20% at IF = ±5mA, VCC = 5V)\n- High input-output isolation voltage (VISO = 3,000VRMS)\n- Non-saturated Response time (tr: typ. 2μs at VCC = 10V, IC = 2mA, RL= 100Ω)\n- CMR 10 kV/μs (typical)"
 		(exclude_from_sim no)
 		(at 140.97 62.23 0)
