File: MotorSheet.kicad_sch (KiCad schematic)
At the start: 27 parts, among them J6 Conn_01x02, J7 Conn_01x02, J8 Conn_01x02, U2 DRV8872DDA, U3 DRV8872DDA, U4 DRV8872DDA

Commit message: Update PDF shematic
Other:
- company: (none) -> MASTODONTE
- title: BR-MOTOR : GPIO Sheet -> BR-MOTOR : MOTOR Sheet
Changed lines of the file:
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@@
 	(paper "A4")
 	(title_block
-		(title "BR-MOTOR : GPIO Sheet")
+		(title "BR-MOTOR : MOTOR Sheet")
 		(date "2025-02-23")
 		(rev "V°1")
+		(company "MASTODONTE")
+		(comment 1 "Paul Miailhe")
 	)
 	(junction
